File: TestCircuit/MorseCodeWatch.sch (KiCad schematic (older format))
At the start: 45 parts, among them J1 USB_B_Micro, J2 Conn_01x02_Male LiPo Battery, J4 Conn_01x03, J5 Conn_01x03, J6 Conn_01x04_Female, SW1 SW_DIP_x01, U1 MCP73831-2-OT, U2 STM32F101CBTx, U3 CAT24C256, U4 NRF51822_MODULE_MDBT40, U5 MIC5225-3.3, U6 AT42QT1010-TSHR, Y1 32.768kHz (535-9166-2-ND)

Commit message: adding correct ground
Parts:
- C1, C2, C7: symbol Device:C -> MorseCodeWatch-rescue:C-Device
- D1, D2, D3, D4: symbol Device:LED -> MorseCodeWatch-rescue:LED-Device
- D5, D6, D7, D8, D9: symbol Diode:1N4148 -> MorseCodeWatch-rescue:1N4148-Diode
- J1: symbol Connector:USB_B_Micro -> MorseCodeWatch-rescue:USB_B_Micro-Connector
- J2: symbol Connector:Conn_01x02_Male -> MorseCodeWatch-rescue:Conn_01x02_Male-Connector
- J4, J5: symbol Connector_Generic:Conn_01x03 -> MorseCodeWatch-rescue:Conn_01x03-Connector_Generic
- J6: symbol Connector:Conn_01x04_Female -> MorseCodeWatch-rescue:Conn_01x04_Female-Connector
- R1, R10, R2, R3, R4, R5: symbol Device:R -> MorseCodeWatch-rescue:R-Device
- SW1: symbol Switch:SW_DIP_x01 -> MorseCodeWatch-rescue:SW_DIP_x01-Switch
- U1: symbol Battery_Management:MCP73831-2-OT -> MorseCodeWatch-rescue:MCP73831-2-OT-Battery_Management
- U2: symbol MCU_ST_STM32F1:STM32F101CBTx -> MorseCodeWatch-rescue:STM32F101CBTx-MCU_ST_STM32F1
- U3: symbol Memory_EEPROM:CAT24C256 -> MorseCodeWatch-rescue:CAT24C256-Memory_EEPROM
- U6: symbol Sensor_Touch:AT42QT1010-TSHR -> MorseCodeWatch-rescue:AT42QT1010-TSHR-Sensor_Touch
Changed lines of the file:
@@
 $EndDescr
 $Comp
-L Connector:USB_B_Micro J1
+L MorseCodeWatch-rescue:USB_B_Micro-Connector J1
 U 1 1 5E4DA130
 P 3650 6950
@@
 $EndComp
 $Comp
-L Device:LED D2
+L MorseCodeWatch-rescue:LED-Device D2
 U 1 1 5E4DDC6D
 P 4900 7500
@@
 $EndComp
 $Comp
-L Device:C C1
+L MorseCodeWatch-rescue:C-Device C1
 U 1 1 5E4DEB11
 P 4400 7000
@@
 $EndComp
 $Comp
-L Device:R R1
+L MorseCodeWatch-rescue:R-Device R1
 U 1 1 5E4E11CC
 P 5200 6950
@@
 $EndComp
 $Comp
-L Device:R R2
+L MorseCodeWatch-rescue:R-Device R2
 U 1 1 5E4E21A5
 P 5200 7500
@@
 $EndComp
 $Comp
-L Device:R R3
+L MorseCodeWatch-rescue:R-Device R3
 U 1 1 5E4E302C
 P 5700 7700
@@
 $EndComp
 $Comp
-L Battery_Management:MCP73831-2-OT U1
+L MorseCodeWatch-rescue:MCP73831-2-OT-Battery_Management U1
 U 1 1 5E4E5A4D
 P 5900 7050
@@
 $EndComp
 $Comp
-L Device:LED D1
+L MorseCodeWatch-rescue:LED-Device D1
 U 1 1 5E4DD022
 P 4900 6950
@@
 	4750 6750 5900 6750
 $Comp
-L power:GND #PWR0101
+L MorseCodeWatch-rescue:GND-power #PWR0101
 U 1 1 5E522086
 P 4400 7800
@@
 $EndComp
 $Comp
-L power:GND #PWR0102
+L MorseCodeWatch-rescue:GND-power #PWR0102
 U 1 1 5E5235BF
 P 4700 7800
@@
 $EndComp
 $Comp
-L power:GND #PWR0103
+L MorseCodeWatch-rescue:GND-power #PWR0103
 U 1 1 5E52368F
 P 6500 7800
@@
 $EndComp
 $Comp
-L power:GND #PWR0104
+L MorseCodeWatch-rescue:GND-power #PWR0104
 U 1 1 5E5236C3
 P 7250 7800
@@
 $EndComp
 $Comp
-L power:GND #PWR0105
+L MorseCodeWatch-rescue:GND-power #PWR0105
 U 1 1 5E52612F
 P 3650 7800
@@
 	5900 7350 5900 7700
 $Comp
-L Connector:Conn_01x02_Male J2
+L MorseCodeWatch-rescue:Conn_01x02_Male-Connector J2
 U 1 1 5E52E8A2
 P 8150 6950
@@
 	7250 5450 7250 5350
 $Comp
-L power:GND #PWR0107
+L MorseCodeWatch-rescue:GND-power #PWR0107
 U 1 1 5E546EB1
 P 11100 6550
@@
 PROG
 $Comp
-L Connector:Conn_01x04_Female J6
+L MorseCodeWatch-rescue:Conn_01x04_Female-Connector J6
 U 1 1 5E58E21D
 P 1350 7650
@@
 SDA
 $Comp
-L Memory_EEPROM:CAT24C256 U3
+L MorseCodeWatch-rescue:CAT24C256-Memory_EEPROM U3
 U 1 1 5E5BF4CC
 P 9400 6750
@@
 	9400 6450 9200 6450
 $Comp
-L Device:R R5
+L MorseCodeWatch-rescue:R-Device R5
 U 1 1 5E5CE454
 P 9700 6450
@@
 $EndComp
 $Comp
-L Device:R R4
+L MorseCodeWatch-rescue:R-Device R4
 U 1 1 5E5CFD10
 P 9700 6350
@@
 	9350 4850 9350 4350
 $Comp
-L MCU_ST_STM32F1:STM32F101CBTx U2
+L MorseCodeWatch-rescue:STM32F101CBTx-MCU_ST_STM32F1 U2
 U 1 1 5E5391EB
 P 9550 5450
@@
 VBAT
 $Comp
-L Connector_Generic:Conn_01x03 J4
+L MorseCodeWatch-rescue:Conn_01x03-Connector_Generic J4
 U 1 1 5E766726
 P 10400 4000
@@
 SWCLK
 $Comp
-L Switch:SW_DIP_x01 SW1
+L MorseCodeWatch-rescue:SW_DIP_x01-Switch SW1
 U 1 1 5EA3EDA2
 P 7250 6400
@@
 	6800 7100 6800 6950
 $Comp
-L power:GND #PWR0106
+L MorseCodeWatch-rescue:GND-power #PWR0106
 U 1 1 5E52A908
 P 6800 7800
@@
 $EndComp
 $Comp
-L Device:C C2
+L MorseCodeWatch-rescue:C-Device C2
 U 1 1 5E4E0C5A
 P 6800 7250
@@
 $EndComp
 $Comp
-L Diode:1N4148 D6
+L MorseCodeWatch-rescue:1N4148-Diode D6
 U 1 1 5EB310A8
 P 9400 2700
@@
 $EndComp
 $Comp
-L Device:LED D3
+L MorseCodeWatch-rescue:LED-Device D3
 U 1 1 5EBDB4CC
 P 7650 2300
@@
 $EndComp
 $Comp
-L Device:LED D4
+L MorseCodeWatch-rescue:LED-Device D4
 U 1 1 5EBE6B40
 P 8050 2300
@@
 Connection ~ 9750 2700
 $Comp
-L Diode:1N4148 D8
+L MorseCodeWatch-rescue:1N4148-Diode D8
 U 1 1 5EB481F6
 P 9400 3300
@@
 $EndComp
 $Comp
-L Diode:1N4148 D7
+L MorseCodeWatch-rescue:1N4148-Diode D7
 U 1 1 5EB3C720
 P 9400 3000
@@
 $EndComp
 $Comp
-L Diode:1N4148 D5
+L MorseCodeWatch-rescue:1N4148-Diode D5
 U 1 1 5EAF45E0
 P 9400 2400
@@
 $EndComp
 $Comp
-L Diode:1N4148 D9
+L MorseCodeWatch-rescue:1N4148-Diode D9
 U 1 1 5ECD1C26
 P 900 3050
@@
 Connection ~ 9550 2400
 $Comp
-L Connector_Generic:Conn_01x03 J5
+L MorseCodeWatch-rescue:Conn_01x03-Connector_Generic J5
 U 1 1 5ED492AB
 P 9250 4150
@@
 	2350 4800 2350 5000
 $Comp
-L Device:R R10
+L MorseCodeWatch-rescue:R-Device R10
 U 1 1 5E920FA0
 P 2350 5150
@@
 TOG-AHLB
 $Comp
-L Device:C C7
+L MorseCodeWatch-rescue:C-Device C7
 U 1 1 5E9084D6
 P 1950 5150
@@
 	1000 4800 850  4800
 $Comp
-L Sensor_Touch:AT42QT1010-TSHR U6
+L MorseCodeWatch-rescue:AT42QT1010-TSHR-Sensor_Touch U6
 U 1 1 5E83AF66
 P 1400 4700
