File: NRF52 MorseCodeWatch/nrf52832_qfaa-SchDoc.sch (KiCad schematic (older format))
At the start: 25 parts, among them J1 Conn_01x04, U1 NRF52832-QFAA-R, U2 AT42QT1010-TSHR, U3 CAT24C256, X1 32mHz, X2 32.768kHz

Commit message: adding correct ground
Parts:
- removed C15: 22pF, symbol Device:C
- removed R1: 1K, symbol Device:R
- removed R2, R3: 10K, symbol Device:R
- removed U3: CAT24C256, symbol Memory_EEPROM:CAT24C256
- removed X1: 32mHz, Crystal:Crystal_SMD_3225-4Pin_3.2x2.5mm_HandSoldering, symbol Device:Crystal
- added C15: 22pF, Capacitor_SMD:C_0402_1005Metric, symbol nrf52832_qfaa-SchDoc-rescue:C-Device
- added C16, C17: C 10uf, Capacitor_SMD:C_0402_1005Metric, symbol MorseCodeWatch-rescue:C-Device
- added D1: LED RED, LED_SMD:LED_0603_1608Metric, symbol MorseCodeWatch-rescue:LED-Device
- added D2: LED GREEN, LED_SMD:LED_0603_1608Metric, symbol MorseCodeWatch-rescue:LED-Device
- added J2: USB_B_Micro, Connector_USB:USB_Micro-B_Wuerth_629105150521, symbol MorseCodeWatch-rescue:USB_B_Micro-Connector
- added J3: Conn_01x02_Male LiPo Battery, Connector_JST:JST_ACH_BM02B-ACHSS-GAN-ETF_1x02-1MP_P1.20mm_Vertical, symbol MorseCodeWatch-rescue:Conn_01x02_Male-Connector
- added M1, M2: Motor_DC, Connector_JST:JST_ACH_BM02B-ACHSS-GAN-ETF_1x02-1MP_P1.20mm_Vertical, symbol Default:Motor_DC
- added R1: 1K, Resistor_SMD:R_0402_1005Metric, symbol nrf52832_qfaa-SchDoc-rescue:R-Device
- added R2, R3: 10K, Resistor_SMD:R_0402_1005Metric, symbol nrf52832_qfaa-SchDoc-rescue:R-Device
- added R4, R5: R, Resistor_SMD:R_0402_1005Metric, symbol MorseCodeWatch-rescue:R-Device
- added R6: R 10K, Resistor_SMD:R_0402_1005Metric, symbol MorseCodeWatch-rescue:R-Device
- added SW1: SW_DIP_x01, Button_Switch_SMD:SW_DIP_SPSTx01_Slide_Copal_CHS-01A_W5.08mm_P1.27mm_JPin, symbol MorseCodeWatch-rescue:SW_DIP_x01-Switch
- added U3: CAT24C256, Package_SO:SOIC-8_3.9x4.9mm_P1.27mm, symbol nrf52832_qfaa-SchDoc-rescue:CAT24C256-Memory_EEPROM
- added U4: MCP73831-2-OT, Package_TO_SOT_SMD:SOT-23-5, symbol MorseCodeWatch-rescue:MCP73831-2-OT-Battery_Management
- added U5: DRV8836, Package_SON:WSON-12-1EP_3x2mm_P0.5mm_EP1x2.65, symbol drv883x:DRV8836
- added X1: 32mHz, symbol nrf52832_qfaa-SchDoc-rescue:Crystal-Device4
- C1, C10, C11, C12, C13, C14, C2, C3, C4, C5, C6, C7, C8, C9: symbol Device:C -> nrf52832_qfaa-SchDoc-rescue:C-Device
- J1: symbol Connector_Generic:Conn_01x04 -> nrf52832_qfaa-SchDoc-rescue:Conn_01x04-Connector_Generic
- L1: symbol pspice:INDUCTOR -> nrf52832_qfaa-SchDoc-rescue:INDUCTOR-pspice
- U1: symbol MCU_Nordic:NRF52832-QFAA-R -> nrf52832_qfaa-SchDoc-rescue:NRF52832-QFAA-R-MCU_Nordic
- U2: symbol Sensor_Touch:AT42QT1010-TSHR -> nrf52832_qfaa-SchDoc-rescue:AT42QT1010-TSHR-Sensor_Touch
- X2: symbol Device:Crystal -> nrf52832_qfaa-SchDoc-rescue:Crystal-Device
Connections:
- net labels added: Motor1, Motor1_out, Motor1_outB, Motor2, Motor2_out, Motor2_outB, Motor_Sleep, PROG, SCL, SDA, STAT, ThermalGND, VBAT-IN, VCC
- wire segments 114 -> 163

Commit message: minor fixes
minor layout changes to pcb
Parts:
- added C18: C 10uf, Capacitor_SMD:C_0402_1005Metric, symbol MorseCodeWatch-rescue:C-Device
- R4, R5: value R -> R 47Ω
Connections:
- net P0.12 is gone; now on net Motor_Sleep: U1.15 (P0.12)
- net GND: now also C18.1; no longer M1.2 (-), M2.2 (-), U5.11 (MODE), U5.7 (BIN2), U5.9 (AIN2)
- net Motor1_outB: now also M1.2 (-)
- net Motor2_outB: now also M2.2 (-)
- net Motor_Sleep: no longer U1.16 (P0.13)
- net VDD_nRF: now also C18.2
- net Motor1 renamed Motor1_ENBL
- net Motor1_ENBL: now also U5.9 (AIN2); no longer U5.10 (AIN1)
- net Motor2 renamed Motor2_ENBL
- net Motor2_ENBL: now also U5.7 (BIN2); no longer U5.8 (BIN1)
- new net Motor1_PHASE: U5.10 (AIN1)
- new net Motor2_PHASE: U5.8 (BIN1)
- new net Motor_Mode: U1.16 (P0.13), U5.11 (MODE)
Changed lines of the file:
@@
 P 3450 2950
 F 0 "R4" H 3520 2996 50  0000 L CNN
-F 1 "R" H 3520 2905 50  0000 L CNN
+F 1 "R 47Ω" H 3520 2905 50  0000 L CNN
 F 2 "Resistor_SMD:R_0402_1005Metric" V 3380 2950 50  0001 C CNN
 F 3 "~" H 3450 2950 50  0001 C CNN
@@
 P 3450 3500
 F 0 "R5" H 3520 3546 50  0000 L CNN
-F 1 "R" H 3520 3455 50  0000 L CNN
+F 1 "R 47Ω" H 3520 3455 50  0000 L CNN
 F 2 "Resistor_SMD:R_0402_1005Metric" V 3380 3500 50  0001 C CNN
 F 3 "~" H 3450 3500 50  0001 C CNN
@@
 	7450 6950 7400 6950
 Text Label 4950 9450 2    50   ~ 0
-GND
+Motor_Mode
 Text Label 7850 9400 0    50   ~ 0
 Motor2_out
@@
 Motor1_out
 Text Label 4950 8950 2    50   ~ 0
-Motor1
+Motor1_PHASE
 Text Label 4950 9200 2    50   ~ 0
-Motor2
+Motor2_PHASE
 Text Label 6350 9200 0    50   ~ 0
 Motor2_out
@@
 Wire Wire Line
 	7350 9400 7150 9400
-Text Label 7150 9400 0    50   ~ 0
-GND
-Text Label 7150 8850 0    50   ~ 0
-GND
+Text Label 7150 9400 2    50   ~ 0
+Motor2_outB
+Text Label 7150 8850 2    50   ~ 0
+Motor1_outB
 Wire Wire Line
 	7350 8850 7150 8850
@@
 Wire Wire Line
 	7400 6750 7450 6750
-Text Label 7150 7650 2    50   ~ 0
-MainSwitch
-Wire Wire Line
-	7400 7650 7150 7650
 Text Label 7100 7450 2    50   ~ 0
-Motor1
+Motor1_ENBL
 Text Label 7100 7550 2    50   ~ 0
-Motor2
-Text Label 7200 7350 2    50   ~ 0
+Motor2_ENBL
+Text Label 7200 7250 2    50   ~ 0
 Motor_Sleep
 Wire Wire Line
 	7100 7450 7400 7450
 Wire Wire Line
-	7400 7350 7200 7350
+	7400 7250 7200 7250
 Wire Wire Line
 	7400 7550 7100 7550
@@
 Motor2_outB
 Text Label 4950 9300 2    50   ~ 0
-GND
+Motor2_ENBL
 Text Label 4950 9050 2    50   ~ 0
-GND
+Motor1_ENBL
 Text Label 4950 9550 2    50   ~ 0
 Motor_Sleep
@@
 Text Label 5700 8700 0    50   ~ 0
 VDD_nRF
+Text Label 7150 7350 2    50   ~ 0
+Motor_Mode
+Wire Wire Line
+	7400 7650 7150 7650
+Text Label 7150 7650 2    50   ~ 0
+MainSwitch
+Wire Wire Line
+	7400 7350 7150 7350
+$Comp
+L MorseCodeWatch-rescue:C-Device C18
+U 1 1 5EE48B3B
+P 5550 8300
+F 0 "C18" H 5665 8346 50  0000 L CNN
+F 1 "C 10uf" H 5665 8255 50  0000 L CNN
+F 2 "Capacitor_SMD:C_0402_1005Metric" H 5588 8150 50  0001 C CNN
+F 3 "~" H 5550 8300 50  0001 C CNN
+	1    5550 8300
+	0    -1   -1   0
+$EndComp
+Wire Wire Line
+	5700 8700 5700 8300
+Wire Wire Line
+	5400 8300 5050 8300
+Text Label 5050 8300 0    50   ~ 0
+GND
 $EndSCHEMATC

Commit message: update PCB with voltage regulator
using a voltage regulator now with the PCB design.

update BOM
Parts:
- removed J1: Conn_01x04, Connector_PinHeader_1.27mm:PinHeader_1x04_P1.27mm_Vertical_SMD_Pin1Right, symbol nrf52832_qfaa-SchDoc-rescue:Conn_01x04-Connector_Generic
- added C19: C 1uf, Capacitor_SMD:C_0402_1005Metric, symbol nrf52832_qfaa-SchDoc-rescue:C-Device-MorseCodeWatch-rescue
- added C20: C 2.2uf, Capacitor_SMD:C_0402_1005Metric, symbol nrf52832_qfaa-SchDoc-rescue:C-Device-MorseCodeWatch-rescue
- added J1: Conn_02x05_Odd_Even, symbol Connector_Generic:Conn_02x05_Odd_Even
- added J5: Battery_Cell, Battery:BatteryHolder_Keystone_3034_1x20mm, symbol Device:Battery_Cell
- added J6: Conn_01x02_Male LiPo Battery, Connector_JST:JST_ACH_BM02B-ACHSS-GAN-ETF_1x02-1MP_P1.20mm_Vertical, symbol nrf52832_qfaa-SchDoc-rescue:Conn_01x02_Male-Connector-MorseCodeWatch-rescue
- added U6: TPS783, Package_TO_SOT_SMD:SOT-23-5, symbol Regulator_Linear:TPS79333-EP
- C16, C17, C18: symbol MorseCodeWatch-rescue:C-Device -> nrf52832_qfaa-SchDoc-rescue:C-Device-MorseCodeWatch-rescue
- D1, D2: symbol MorseCodeWatch-rescue:LED-Device -> nrf52832_qfaa-SchDoc-rescue:LED-Device-MorseCodeWatch-rescue
- J2: symbol MorseCodeWatch-rescue:USB_B_Micro-Connector -> nrf52832_qfaa-SchDoc-rescue:USB_B_Micro-Connector-MorseCodeWatch-rescue
- J3: symbol MorseCodeWatch-rescue:Conn_01x02_Male-Connector -> nrf52832_qfaa-SchDoc-rescue:Conn_01x02_Male-Connector-MorseCodeWatch-rescue
- M1, M2: symbol Default:Motor_DC -> nrf52832_qfaa-SchDoc-rescue:Motor_DC-Default
- R4, R5, R6: symbol MorseCodeWatch-rescue:R-Device -> nrf52832_qfaa-SchDoc-rescue:R-Device-MorseCodeWatch-rescue
- SW1: symbol MorseCodeWatch-rescue:SW_DIP_x01-Switch -> nrf52832_qfaa-SchDoc-rescue:SW_DIP_x01-Switch-MorseCodeWatch-rescue
- U4: symbol MorseCodeWatch-rescue:MCP73831-2-OT-Battery_Management -> nrf52832_qfaa-SchDoc-rescue:MCP73831-2-OT-Battery_Management-MorseCodeWatch-rescue
Connections:
- net GND: now also C19.2, C20.2, J1.3 (Pin_3), J1.5 (Pin_5), J5.2 (-), U6.2 (GND), U6.4 (BP); no longer J3.2 (Pin_2)
- net Motor1_out: now also J6.1 (Pin_1)
- net Motor1_outB: now also J6.2 (Pin_2)
- net P0.21: now also J1.10 (Pin_10)
- net SWDCLK: now also J1.4 (Pin_4)
- net SWDIO: now also J1.2 (Pin_2)
- net TouchPad: now also J3.1 (Pin_1), J3.2 (Pin_2)
- net VBAT-IN: now also J5.1 (+); no longer J3.1 (Pin_1)
- net VDD_nRF: now also C20.1, J1.1 (Pin_1), U6.5 (OUT); no longer SW1.2
- new net VDD_in: C19.1, SW1.2, U6.1 (IN), U6.3 (EN)
Other:
- moved on the sheet: J3
